Commit message: Updated materials file

File: urdf/fura2a.xacro (robot description, xacro)
@@ -15,5 +15,5 @@
       <mesh filename="file://$(find fura2a)/meshes/base_link.stl" scale="0.001 0.001 0.001"/>
     </geometry>
-    <material name="silver"/>
+    <material name="CustomRed"/>
   </visual>
   <collision>
@@ -35,5 +35,5 @@
       <mesh filename="file://$(find fura2a)/meshes/column.stl" scale="0.001 0.001 0.001"/>
     </geometry>
-    <material name="silver"/>
+    <material name="CustomYellow"/>
   </visual>
   <collision>
@@ -55,5 +55,5 @@
       <mesh filename="file://$(find fura2a)/meshes/arm.stl" scale="0.001 0.001 0.001"/>
     </geometry>
-    <material name="silver"/>
+    <material name="CustomGreen"/>
   </visual>
   <collision>
@@ -75,5 +75,5 @@
       <mesh filename="file://$(find fura2a)/meshes/pendulum.stl" scale="0.001 0.001 0.001"/>
     </geometry>
-    <material name="silver"/>
+    <material name="CUstomBlue"/>
   </visual>
   <collision>

File: urdf/materials.xacro (robot description, xacro)
@@ -1,6 +1,29 @@
-<?xml version="1.0" ?>
-<robot name="fura2a" xmlns:xacro="http://www.ros.org/wiki/xacro" >
-<material name="silver">
-  <color rgba="0.700 0.700 0.700 1.000"/>
-</material>
+<?xml version="1.0"?>
+<robot xmlns:xacro="http://www.ros.org/wiki/xacro" name="materials">
+  <!-- Define custom materials -->
+  <!-- Silver Material -->
+  <material name="Silver">
+    <color rgba="0.75 0.75 0.75 1.0"/>
+  </material>
+  <!-- Custom Red Material -->
+  <material name="CustomRed">
+    <color rgba="1 0 0 1"/>
+  </material>
+  <!-- Custom Green Material -->
+  <material name="CustomGreen">
+    <color rgba="0 1 0 1"/>
+  </material>
+  <!-- Custom Blue Material -->
+  <material name="CustomBlue">
+    <color rgba="0 0 1 1"/>
+  </material>
+  <!-- Custom Yellow Material -->
+  <material name="CustomYellow">
+    <color rgba="1 1 0 1"/>
+  </material>
+  <!-- Custom Purple Material -->
+  <material name="CustomPurple">
+    <color rgba="0.5 0 0.5 1"/>
+  </material>
+  <!-- Add more materials as needed -->
 </robot>

Commit message: Updated materials files

File: urdf/fura2a.xacro (robot description, xacro)
@@ -75,5 +75,5 @@
       <mesh filename="file://$(find fura2a)/meshes/pendulum.stl" scale="0.001 0.001 0.001"/>
     </geometry>
-    <material name="CUstomBlue"/>
+    <material name="CustomBlue"/>
   </visual>
   <collision>

Commit message: added swingup and lqr basis

File: urdf/fura2a.xacro (robot description, xacro)
@@ -66,5 +66,5 @@
 <link name="pendulum">
   <inertial>
-    <origin xyz="0.0049999999999999906 1.2138781501420367e-17 0.059999999999999915" rpy="0 0 0"/>
+    <origin xyz="0.005 1.2138781501420367e-17 0.06" rpy="0 0 0"/>
     <mass value="0.08939794594871456"/>
     <inertia ixx="0.000157" iyy="0.000157" izz="1e-06" ixy="0.0" iyz="-0.0" ixz="-0.0"/>
@@ -96,5 +96,5 @@
 </joint>
 <joint name="pendulum_joint" type="continuous">
-  <origin xyz="0.075 0.0 0.0125" rpy="0 0 0"/>
+  <origin xyz="0.075 0.0 0.0125" rpy="-3.1415926 0 0"/>
   <parent link="arm"/>
   <child link="pendulum"/>

Commit message: general update

File: urdf/fura2a.xacro (robot description, xacro)
@@ -46,19 +46,19 @@
 <link name="arm">
   <inertial>
-    <origin xyz="0.007967562168493848 3.0890324677637924e-17 0.012500000000000011" rpy="0 0 0"/>
-    <mass value="1.786614971490255"/>
-    <inertia ixx="0.001119" iyy="0.001785" izz="0.002717" ixy="-0.0" iyz="0.0" ixz="-0.0"/>
+    <origin xyz="0.026682566071217124 -3.832567320079414e-17 0.014261674729385443" rpy="0 0 0"/>
+    <mass value="0.5334931362492104"/>
+    <inertia ixx="0.000381" iyy="0.000781" izz="0.001096" ixy="-0.0" iyz="-0.0" ixz="2.5e-05"/>
   </inertial>
   <visual>
     <origin xyz="-0.0 -0.0 -0.145" rpy="0 0 0"/>
     <geometry>
-      <mesh filename="file://$(find fura2a)/meshes/arm.stl" scale="0.001 0.001 0.001"/>
+      <mesh filename="file://$(find fura2a)/meshes/hollowed_arm.stl" scale="0.001 0.001 0.001"/>
     </geometry>
-    <material name="CustomGreen"/>
+    <material name="silver"/>
   </visual>
   <collision>
     <origin xyz="-0.0 -0.0 -0.145" rpy="0 0 0"/>
     <geometry>
-      <mesh filename="file://$(find fura2a)/meshes/arm.stl" scale="0.001 0.001 0.001"/>
+      <mesh filename="file://$(find fura2a)/meshes/hollowed_arm.stl" scale="0.001 0.001 0.001"/>
     </geometry>
   </collision>
@@ -66,19 +66,19 @@
 <link name="pendulum">
   <inertial>
-    <origin xyz="0.005 1.2138781501420367e-17 0.06" rpy="0 0 0"/>
+    <origin xyz="0.0049999999999999906 -7.34788079488412e-18 -0.05999999999999997" rpy="0 0 0"/>
     <mass value="0.08939794594871456"/>
-    <inertia ixx="0.000157" iyy="0.000157" izz="1e-06" ixy="0.0" iyz="-0.0" ixz="-0.0"/>
+    <inertia ixx="0.000157" iyy="0.000157" izz="1e-06" ixy="0.0" iyz="-0.0" ixz="0.0"/>
   </inertial>
   <visual>
     <origin xyz="-0.075 -0.0 -0.1575" rpy="0 0 0"/>
     <geometry>
-      <mesh filename="file://$(find fura2a)/meshes/pendulum.stl" scale="0.001 0.001 0.001"/>
+      <mesh filename="file://$(find fura2a)/meshes/pendulum_down.stl" scale="0.001 0.001 0.001"/>
     </geometry>
-    <material name="CustomBlue"/>
+    <material name="silver"/>
   </visual>
   <collision>
     <origin xyz="-0.075 -0.0 -0.1575" rpy="0 0 0"/>
     <geometry>
-      <mesh filename="file://$(find fura2a)/meshes/pendulum.stl" scale="0.001 0.001 0.001"/>
+      <mesh filename="file://$(find fura2a)/meshes/pendulum_down.stl" scale="0.001 0.001 0.001"/>
     </geometry>
   </collision>
@@ -94,10 +94,12 @@
   <child link="arm"/>
   <axis xyz="0.0 0.0 1.0"/>
+  <dynamics damping="0.01" friction="0.0"/> <!-- Added damping -->
 </joint>
 <joint name="pendulum_joint" type="continuous">
-  <origin xyz="0.075 0.0 0.0125" rpy="-3.1415926 0 0"/>
+  <origin xyz="0.075 0.0 0.0125" rpy="0 0 0"/>
   <parent link="arm"/>
   <child link="pendulum"/>
   <axis xyz="1.0 0.0 0.0"/>
+  <dynamics damping="0.05" friction="0.0"/> <!-- Added damping -->
 </joint>
 </robot>

Commit message: tried adding fake arm

File: urdf/fura2a.xacro (robot description, xacro)
@@ -46,19 +46,19 @@
 <link name="arm">
   <inertial>
-    <origin xyz="0.026682566071217124 -3.832567320079414e-17 0.014261674729385443" rpy="0 0 0"/>
-    <mass value="0.5334931362492104"/>
-    <inertia ixx="0.000381" iyy="0.000781" izz="0.001096" ixy="-0.0" iyz="-0.0" ixz="2.5e-05"/>
+    <origin xyz="0.037500000000000006 -2.220446049250313e-18 0.0062500000000000056" rpy="0 0 0"/>
+    <mass value="0.07359375"/>
+    <inertia ixx="2e-06" iyy="3.5e-05" izz="3.5e-05" ixy="-0.0" iyz="0.0" ixz="0.0"/>
   </inertial>
   <visual>
     <origin xyz="-0.0 -0.0 -0.145" rpy="0 0 0"/>
     <geometry>
-      <mesh filename="file://$(find fura2a)/meshes/hollowed_arm.stl" scale="0.001 0.001 0.001"/>
+      <mesh filename="file://$(find fura2a)/meshes/fake_arm.stl" scale="0.001 0.001 0.001"/>
     </geometry>
-    <material name="silver"/>
+    <material name="Silver"/>
   </visual>
   <collision>
     <origin xyz="-0.0 -0.0 -0.145" rpy="0 0 0"/>
     <geometry>
-      <mesh filename="file://$(find fura2a)/meshes/hollowed_arm.stl" scale="0.001 0.001 0.001"/>
+      <mesh filename="file://$(find fura2a)/meshes/fake_arm.stl" scale="0.001 0.001 0.001"/>
     </geometry>
   </collision>
@@ -66,19 +66,19 @@
 <link name="pendulum">
   <inertial>
-    <origin xyz="0.0049999999999999906 -7.34788079488412e-18 -0.05999999999999997" rpy="0 0 0"/>
-    <mass value="0.08939794594871456"/>
-    <inertia ixx="0.000157" iyy="0.000157" izz="1e-06" ixy="0.0" iyz="-0.0" ixz="0.0"/>
+    <origin xyz="0.0050000000000000044 -8.574075045622943e-18 -0.0675" rpy="0 0 0"/>
+    <mass value="0.10597499999999999"/>
+    <inertia ixx="0.000162" iyy="0.000162" izz="2e-06" ixy="0.0" iyz="-0.0" ixz="-0.0"/>
   </inertial>
   <visual>
-    <origin xyz="-0.075 -0.0 -0.1575" rpy="0 0 0"/>
+    <origin xyz="-0.075 0.0 -0.1575" rpy="0 0 0"/>
     <geometry>
-      <mesh filename="file://$(find fura2a)/meshes/pendulum_down.stl" scale="0.001 0.001 0.001"/>
+      <mesh filename="file://$(find fura2a)/meshes/cuboid_pendulum.stl" scale="0.001 0.001 0.001"/>
     </geometry>
-    <material name="silver"/>
+    <material name="Silver"/>
   </visual>
   <collision>
-    <origin xyz="-0.075 -0.0 -0.1575" rpy="0 0 0"/>
+    <origin xyz="-0.075 0.0 -0.1575" rpy="0 0 0"/>
     <geometry>
-      <mesh filename="file://$(find fura2a)/meshes/pendulum_down.stl" scale="0.001 0.001 0.001"/>
+      <mesh filename="file://$(find fura2a)/meshes/cuboid_pendulum.stl" scale="0.001 0.001 0.001"/>
     </geometry>
   </collision>

Commit message: end of fake arm attempt

File: urdf/fura2a.xacro (robot description, xacro)
@@ -7,5 +7,5 @@
   <inertial>
     <origin xyz="-1.4655194516233777e-17 0.0 0.009896382619700488" rpy="0 0 0"/>
-    <mass value="4.871674272906388"/>
+    <mass value="50"/>
     <inertia ixx="0.012198" iyy="0.012198" izz="0.024075" ixy="-0.0" iyz="0.0" ixz="0.0"/>
   </inertial>
@@ -27,5 +27,5 @@
   <inertial>
     <origin xyz="1.0658141036401502e-16 0.0 0.062495742145380256" rpy="0 0 0"/>
-    <mass value="7.706192602274715"/>
+    <mass value="50"/>
     <inertia ixx="0.014849" iyy="0.014849" izz="0.009632" ixy="0.0" iyz="0.0" ixz="0.0"/>
   </inertial>
@@ -53,7 +53,7 @@
     <origin xyz="-0.0 -0.0 -0.145" rpy="0 0 0"/>
     <geometry>
-      <mesh filename="file://$(find fura2a)/meshes/fake_arm.stl" scale="0.001 0.001 0.001"/>
+      <mesh filename="file://$(find fura2a)/meshes/hollowed_arm.stl" scale="0.001 0.001 0.001"/>
     </geometry>
-    <material name="Silver"/>
+    <material name="CustomGreen"/>
   </visual>
   <collision>
@@ -71,9 +71,9 @@
   </inertial>
   <visual>
-    <origin xyz="-0.075 0.0 -0.1575" rpy="0 0 0"/>
+    <origin xyz="-0.075 -0.0 -0.1575" rpy="0 0 0"/>
     <geometry>
-      <mesh filename="file://$(find fura2a)/meshes/cuboid_pendulum.stl" scale="0.001 0.001 0.001"/>
+      <mesh filename="file://$(find fura2a)/meshes/pendulum_down.stl" scale="0.001 0.001 0.001"/>
     </geometry>
-    <material name="Silver"/>
+    <material name="CustomBlue"/>
   </visual>
   <collision>
@@ -94,5 +94,5 @@
   <child link="arm"/>
   <axis xyz="0.0 0.0 1.0"/>
-  <dynamics damping="0.01" friction="0.0"/> <!-- Added damping -->
+  <dynamics damping="0.0001"/> Added damping
 </joint>
 <joint name="pendulum_joint" type="continuous">
@@ -101,5 +101,5 @@
   <child link="pendulum"/>
   <axis xyz="1.0 0.0 0.0"/>
-  <dynamics damping="0.05" friction="0.0"/> <!-- Added damping -->
+  <dynamics damping="0.0003"/> Added damping
 </joint>
 </robot>

Commit message: time to switch

File: urdf/fura2a.xacro (robot description, xacro)
@@ -44,9 +44,29 @@
   </collision>
 </link>
-<link name="arm">
+<!-- <link name="arm">
   <inertial>
     <origin xyz="0.037500000000000006 -2.220446049250313e-18 0.0062500000000000056" rpy="0 0 0"/>
     <mass value="0.07359375"/>
     <inertia ixx="2e-06" iyy="3.5e-05" izz="3.5e-05" ixy="-0.0" iyz="0.0" ixz="0.0"/>
+  </inertial>
+  <visual>
+    <origin xyz="-0.0 -0.0 -0.145" rpy="0 0 0"/>
+    <geometry>
+      <mesh filename="file://$(find fura2a)/meshes/hollowed_arm.stl" scale="0.001 0.001 0.001"/>
+    </geometry>
+    <material name="CustomGreen"/>
+  </visual>
+  <collision>
+    <origin xyz="-0.0 -0.0 -0.145" rpy="0 0 0"/>
+    <geometry>
+      <mesh filename="file://$(find fura2a)/meshes/fake_arm.stl" scale="0.001 0.001 0.001"/>
+    </geometry>
+  </collision>
+</link> -->
+<link name="arm">
+  <inertial>
+    <origin xyz="0.037500000000000006 -2.220446049250313e-18 0.0062500000000000056" rpy="0 0 0"/>
+    <mass value="0.3"/>
+    <inertia ixx="8.15286624e-06" iyy="1.42675159e-04" izz="1.42675159e-04" ixy="-0.0" iyz="0.0" ixz="0.0"/>
   </inertial>
   <visual>
@@ -94,5 +114,5 @@
   <child link="arm"/>
   <axis xyz="0.0 0.0 1.0"/>
-  <dynamics damping="0.0001"/> Added damping
+  <!-- <dynamics damping="0.0001"/> Added damping -->
 </joint>
 <joint name="pendulum_joint" type="continuous">
@@ -101,5 +121,5 @@
   <child link="pendulum"/>
   <axis xyz="1.0 0.0 0.0"/>
-  <dynamics damping="0.0003"/> Added damping
+  <!-- <dynamics damping="0.0003"/> Added damping -->
 </joint>
 </robot>

Commit message: fixed material

File: urdf/fura2a.xacro (robot description, xacro)
@@ -55,5 +55,5 @@
       <mesh filename="file://$(find fura2a)/meshes/hollowed_arm.stl" scale="0.001 0.001 0.001"/>
     </geometry>
-    <material name="silver"/>
+    <material name="Silver"/>
   </visual>
   <collision>
@@ -75,5 +75,5 @@
       <mesh filename="file://$(find fura2a)/meshes/pendulum_down.stl" scale="0.001 0.001 0.001"/>
     </geometry>
-    <material name="silver"/>
+    <material name="Silver"/>
   </visual>
   <collision>

Commit message: changed swingup function slightly

File: urdf/fura2a.xacro (robot description, xacro)
@@ -44,5 +44,5 @@
   </collision>
 </link>
-<link name="arm">
+<!-- <link name="arm">
   <inertial>
     <origin xyz="0.007967562168493848 3.0890324677637924e-17 0.012500000000000011" rpy="0 0 0"/>
@@ -61,4 +61,24 @@
     <geometry>
       <mesh filename="file://$(find fura2a)/meshes/arm.stl" scale="0.001 0.001 0.001"/>
+    </geometry>
+  </collision>
+</link> -->
+<link name="arm">
+  <inertial>
+    <origin xyz="0.026682566071217124 -3.832567320079414e-17 0.014261674729385443" rpy="0 0 0"/>
+    <mass value="0.5334931362492104"/>
+    <inertia ixx="0.000381" iyy="0.000781" izz="0.001096" ixy="-0.0" iyz="-0.0" ixz="2.5e-05"/>
+  </inertial>
+  <visual>
+    <origin xyz="-0.0 -0.0 -0.145" rpy="0 0 0"/>
+    <geometry>
+      <mesh filename="file://$(find fura2a)/meshes/hollowed_arm.stl" scale="0.001 0.001 0.001"/>
+    </geometry>
+    <material name="silver"/>
+  </visual>
+  <collision>
+    <origin xyz="-0.0 -0.0 -0.145" rpy="0 0 0"/>
+    <geometry>
+      <mesh filename="file://$(find fura2a)/meshes/hollowed_arm.stl" scale="0.001 0.001 0.001"/>
     </geometry>
   </collision>

Commit message: jhk

File: urdf/fura2a.xacro (robot description, xacro)
@@ -75,5 +75,5 @@
       <mesh filename="file://$(find fura2a)/meshes/hollowed_arm.stl" scale="0.001 0.001 0.001"/>
     </geometry>
-    <material name="silver"/>
+    <material name="Silver"/>
   </visual>
   <collision>
@@ -104,4 +104,24 @@
   </collision>
 </link>
+<!-- <link name="pendulum">
+  <inertial>
+    <origin xyz="0.005 1.2138781501420367e-17 0.06" rpy="0 0 0"/>
+    <mass value="0.08939794594871456"/>
+    <inertia ixx="0.000157" iyy="0.000157" izz="1e-06" ixy="0.0" iyz="-0.0" ixz="-0.0"/>
+  </inertial>
+  <visual>
+    <origin xyz="-0.075 -0.0 -0.1575" rpy="0 0 0"/>
+    <geometry>
+      <mesh filename="file://$(find fura2a)/meshes/cuboid_pendulum.stl" scale="0.001 0.001 0.001"/>
+    </geometry>
+    <material name="CustomBlue"/>
+  </visual>
+  <collision>
+    <origin xyz="-0.075 -0.0 -0.1575" rpy="0 0 0"/>
+    <geometry>
+      <mesh filename="file://$(find fura2a)/meshes/cuboid_pendulum.stl" scale="0.001 0.001 0.001"/>
+    </geometry>
+  </collision>
+</link> -->
 <joint name="base_column_joint" type="fixed">
   <origin xyz="0.0 0.0 0.02" rpy="0 0 0"/>
@@ -121,3 +141,9 @@
   <axis xyz="1.0 0.0 0.0"/>
 </joint>
+<!-- <joint name="pendulum joint" type="continuous">
+  <origin xyz="0.075 0.0 0.0125" rpy="0 0 0"/>
+  <parent link="arm"/>
+  <child link="pendulum"/>
+  <axis xyz="1.0 0.0 0.0"/>
+</joint> -->
 </robot>
